File: hardware/kicad/front-display-board-rev0-archive/Front display board.kicad_sch (KiCad schematic)
At the start: 18 parts, among them J1 Back of TFT, J2 SD Connection, SW1 RotaryEncoder_Switch, U1 DISP 1, U3 ESP32-C6-DevKitM-Amazon

Commit message: Add files via upload
here is the most recent files
Parts:
- removed C2: 100nF, PCM_JLCPCB:C_0603, symbol PCM_JLCPCB-Capacitors:0603,100nF
- removed C3: 100uF, PCM_JLCPCB:C_1206, symbol PCM_JLCPCB-Capacitors:1206,100uF
- removed H10, H6, H8: VM2, MountingHole:MountingHole_3.5mm, symbol Mechanical:MountingHole
- removed H5, H7, H9: VM1, MountingHole:MountingHole_3.5mm, symbol Mechanical:MountingHole
- removed SW1: RotaryEncoder_Switch, Connector_PinSocket_2.54mm:PinSocket_1x05_P2.54mm_Vertical, symbol Device:RotaryEncoder_Switch
- added 5mm1: ~, 1My_Parts_ Passive:5mm LOGO, symbol 1My_Passive:TNES Logo 5mm
- added C10: 100nF, PCM_JLCPCB:C_0603, symbol PCM_JLCPCB-Capacitors:0603,100nF
- added C4, C5: 10uF, PCM_JLCPCB:C_CASE-A-3216-18(mm), symbol PCM_JLCPCB-Capacitors:CASE-A-3216-18(mm),10uF
- added C6, C7: 100nF, PCM_JLCPCB:C_0805, symbol PCM_JLCPCB-Capacitors:0805,100nF,(2)
- added C8, C9: 330uf, Capacitor_SMD:CP_Elec_6.3x7.7, symbol Device:C_Small_US
- added D1: M1, PCM_JLCPCB:D_SMA, symbol PCM_JLCPCB-Diodes:General,M1
- added D2: RCLAMP0524PATCT, digikey-footprints:UFDFN-10_2.5x1mm, symbol dk_TVS-Diodes:RCLAMP0524PATCT
- added D3: SMAJ5.0A, PCM_JLCPCB:D_SMA, symbol PCM_JLCPCB-Diodes:TVS-Uni,SMAJ5.0A
- added D4: Green, PCM_JLCPCB:D_0805, symbol PCM_JLCPCB-Diodes:LED,0805,Green
- added D5: 1N5819WS, PCM_JLCPCB:D_SOD-323, symbol PCM_JLCPCB-Diodes:Schottky,1N5819WS
- added F1: PTC RESET FUSE 6V 500mA 0805, PCM_JLCPCB:R_0805, symbol Device:Polyfuse
- added J3: 2 x 5 IDE, Connector_IDC:IDC-Header_2x05_P2.54mm_Latch_Vertical, symbol Connector_Generic:Conn_02x05_Odd_Even
- added R1: 10kΩ, PCM_JLCPCB:R_0805, symbol PCM_JLCPCB-Resistors:0805,10kΩ
- added R2: 120Ω, PCM_JLCPCB:R_0805, symbol PCM_JLCPCB-Resistors:0805,120Ω
- added R3, R4: 220Ω, PCM_JLCPCB:R_0805, symbol PCM_JLCPCB-Resistors:0805,220Ω
- added R5: 0Ω, PCM_JLCPCB:R_0805, symbol PCM_JLCPCB-Resistors:0805,0Ω
- added SW2: RotaryEncoder_Switch, Connector_PinHeader_2.54mm:PinHeader_1x05_P2.54mm_Vertical, symbol 1My Basic Componets:RotaryEncoder_Switch
- added TP1, TP10, TP11, TP12, TP13, TP14, TP15, TP16, TP17, TP18, TP19, TP2, TP20, TP21, TP3, TP4, TP5, TP6, TP7, TP8, TP9: 5015, digikey-footprints:Test_Point_2.67x1.02mm, symbol dk_Test-Points:5015
- added U2: AMS1117, PCM_JLCPCB:SOT-223-3_L6.5-W3.4-P2.30-LS7.0-BR, symbol PCM_JLCPCB-Power:LDO, 3.3V, 1A
- U1: footprint Display:hoysond 480 x 320 -> 1My_Parts_ MPUs:Hosyond 4.0 480x320; now left out of the parts list
- U3: now left out of the parts list
Connections:
- net CS (TFT_CS) is gone; now on net CS: J1.3 (Pin_3), U1.3 (~{CS})
- net DC/RS is gone; now on net D/C: J1.5 (Pin_5), U1.5 (D/~{C})
- net SPI SCK is gone; now on net SCLK: J1.10 (Pin_10), J1.7 (Pin_7), U1.10 (T_CLK), U1.7 (SCK)
- net T_CS is gone; now on net Touch CS: J1.11 (Pin_11), U1.11 (T_~CS)
- net T_IRQ is gone; now on net IRQ: J1.14 (Pin_14), U1.14 (T_IRQ)
- net Encoder B: now also U3.28 (GPIO3), SW2.2 (DT)
- net Encoder SW: now also U3.24 (GPIO23), SW2.3 (SW)
- net GND: now also U3.1 (GND), U3.17 (GND), U3.30 (GND), C10.1, C4.2, C5.2, C6.2, C7.2, C8.2, C9.2, D2.3, D2.8, D3.2, J3.1 (Pin_1), J3.3 (Pin_3), J3.7 (Pin_7), R2.2, SW2.5 (GND), TP17.1, U2.1 (GND)
- net RST: now also U3.20 (GPIO19), TP7.1
- net SD card CS: now reaches J2.4 (Pin_4), U1.15 (SD_CS)
- net SD card CS: now also U3.25 (GPIO15), TP13.1
- net MISO: now reaches J2.3 (Pin_3), U1.16 (SD_MOSI)
- net MISO: now also J1.13 (Pin_13), J1.6 (Pin_6), U1.13 (T_DO), U1.6 (MOSI), U3.12 (GPIO11), TP5.1
- net MOSI: now reaches J2.2 (Pin_2), U1.17 (SD_MISO)
- net MOSI: now also J1.12 (Pin_12), J1.9 (Pin_9), U1.12 (T_DIN), U1.9 (MISO), U3.14 (GPIO13), TP11.1
- net SCLK: now reaches J2.1 (Pin_1), U1.18 (SD_SCK)
- net SCLK: now also U3.13 (GPIO12), TP9.1
- net GPIO8: now reaches U3.10 (GPIO8)
- net GPIO8: now also TP18.1
- net CS: now reaches U3.11 (GPIO10)
- net CS: now also TP6.1
- net Vbus: now reaches U3.15 (5V)
- net Vbus: now also U3.16 (5V), D5.2
- net GPIO9: now reaches U3.18 (GPIO9)
- net GPIO9: now also TP19.1
- net D/C: now reaches U3.19 (GPIO18)
- net D/C: now also TP8.1
- net +3V3: now reaches U3.2 (3V3)
- net +3V3: now also C1.2, J1.1 (Pin_1), U1.1 (VCC), C10.2, C4.1, C5.1, C6.1, C9.1, D1.2, D4.2, R1.1, SW2.4 (+V), TP16.1, U2.2 (VOUT), U2.4 (VOUT)
- net PMW: now reaches U3.21 (GPIO20)
- net PMW: now also J1.8 (Pin_8), U1.8 (LED), TP10.1
- net IRQ: now reaches U3.22 (GPIO21)
- net Touch CS: now reaches U3.23 (GPIO22)
- net Touch CS: now also TP12.1
- net Encoder A: now reaches U3.29 (GPIO2)
- net Encoder A: now also SW2.1 (CLK)
- net at U3.3 (EN/RESET): now also R1.2
- net SPI_SCLK: now reaches U3.4 (GPIO4)
- net SPI_SCLK: now also D2.1, J3.4 (Pin_4), TP1.1
- net SPI_MOSI: now reaches U3.5 (GPIO5)
- net SPI_MOSI: now also D2.4, J3.8 (Pin_8), TP2.1
- net SPI_MISO: now reaches U3.6 (GPIO6)
- net SPI_MISO: now also D2.2, J3.6 (Pin_6), TP3.1
- net SPI_CS: now reaches U3.7 (GPIO7)
- net SPI_CS: now also D2.5, J3.10 (Pin_10), TP4.1
- net RTS/CTS: now reaches U3.8 (GPIO0)
- net RTS/CTS: now also R3.2, TP20.1
- net GPIO1: now reaches U3.9 (GPIO1)
- net GPIO1: now also R4.2, TP21.1
- removed net 3v3: C1.2, J1.1 (Pin_1), J1.8 (Pin_8), U1.1 (VCC), U1.8 (LED)
- removed net SPI MISO / SDO : J1.12 (Pin_12), J1.6 (Pin_6), U1.12 (T_DIN), U1.6 (MOSI)
- removed net SPI MOSI / SDI: J1.13 (Pin_13), J1.9 (Pin_9), U1.13 (T_DO), U1.9 (MISO)
- new net: C7.1, C8.1, D1.1, F1.2, R5.2, TP15.1, U2.3 (VIN)
- new net: D4.1, R2.1
- new net: D5.1, R5.1
- new net: J3.9 (Pin_9), R4.1
- new net: J3.5 (Pin_5), R3.1
- new net 5 V_IN: D3.1, F1.1, J3.2 (Pin_2), TP14.1
- no-connect marks 4 -> 6
Other:
- note added: "Input connector"
- note added: "Power Conditioning"
- note added: "TFT (ST7796S) Touch (XPT2046)"
- note added: "To add next rev"
- title: (none) -> 4.0 TFT Display Board  
- moved on the sheet: C1, H1, H2, H3, H4, J1, J2, U1, U3
